Commit message: fix: modify urdf of pro16, pro7, zu18

File: jaka_robot_v2.2/src/jaka_description/urdf/jaka_Pro 7.urdf (robot description, URDF)
Before this commit: robot Pro 7.SLDASM, 8 links, 7 joints
Joints:
- joint joint_1: axis 0 0 -1 -> 0 0 1
- joint joint_5: axis 0 0 -1 -> 0 0 1
- joint joint_6: axis 0 0 -1 -> 0 0 1

File: jaka_robot_v2.2/src/jaka_description/urdf/jaka_pro16.urdf (robot description, URDF)
Before this commit: robot jaka_pro16, 8 links, 7 joints
Joints:
- joint joint_1: axis 0 0 -1 -> 0 0 1
- joint joint_4: axis 0 0 -1 -> 0 0 1
