Commit message: fix: Modify the zu12 URDF

File: jaka_robot_v2.2/src/jaka_description/urdf/jaka_zu12.urdf (robot description, URDF)
Before this commit: robot jaka_zu12, 8 links, 7 joints
Joints:
- joint fixed: origin (none) -> xyz=0 0 0.04 rpy=0 0 0

File: jaka_robot_v2.2/src/jaka_description/urdf/jaka_zu18.urdf (robot description, URDF)
Before this commit: robot jaka_zu18, 8 links, 7 joints
Joints:
- joint fixed: origin (none) -> xyz=0 0 0 rpy=0 0 0

File: jaka_robot_v2.2/src/jaka_description/urdf/jaka_zu3.urdf (robot description, URDF)
Before this commit: robot jaka_zu3, 8 links, 7 joints
Joints:
- joint fixed: origin (none) -> xyz=-0.002 0 -0.00001 rpy=0 0 0

File: jaka_robot_v2.2/src/jaka_description/urdf/jaka_zu5.urdf (robot description, URDF)
Before this commit: robot jaka_zu5, 8 links, 7 joints
Joints:
- joint fixed: origin (none) -> xyz=0 0 0 rpy=0 0 0

File: jaka_robot_v2.2/src/jaka_description/urdf/jaka_zu7.urdf (robot description, URDF)
Before this commit: robot jaka_zu7, 8 links, 7 joints
Joints:
- joint fixed: origin (none) -> xyz=0 0 0 rpy=0 0 0
